Commit message: Fix URDF mesh paths

File: robot/base_fixed.urdf (robot description, URDF)
Before this commit: robot base, 9 links, 8 joints
Links:
- link Base_1: geometry collision mesh filename=../meshes/Base_1.stl scale=0.001 0.001 0.001; visual mesh filename=../meshes/Base_1.stl scale=0.001 0.001 0.001
- link finger1_1: geometry collision mesh filename=../meshes/finger1_1.stl scale=0.001 0.001 0.001; visual mesh filename=../meshes/finger1_1.stl scale=0.001 0.001 0.001
- link finger2_1: geometry collision mesh filename=../meshes/finger2_1.stl scale=0.001 0.001 0.001; visual mesh filename=../meshes/finger2_1.stl scale=0.001 0.001 0.001
- link jaw2_1: geometry collision mesh filename=../meshes/jaw2_1.stl scale=0.001 0.001 0.001; visual mesh filename=../meshes/jaw2_1.stl scale=0.001 0.001 0.001
- link jaw3_1: geometry collision mesh filename=../meshes/jaw3_1.stl scale=0.001 0.001 0.001; visual mesh filename=../meshes/jaw3_1.stl scale=0.001 0.001 0.001
- link jaw4_1: geometry collision mesh filename=../meshes/jaw4_1.stl scale=0.001 0.001 0.001; visual mesh filename=../meshes/jaw4_1.stl scale=0.001 0.001 0.001
- link jaw5_1: geometry collision mesh filename=../meshes/jaw5_1.stl scale=0.001 0.001 0.001; visual mesh filename=../meshes/jaw5_1.stl scale=0.001 0.001 0.001
- link jaw6_1: geometry collision mesh filename=../meshes/jaw6_1.stl scale=0.001 0.001 0.001; visual mesh filename=../meshes/jaw6_1.stl scale=0.001 0.001 0.001
- link jawpart1_1: geometry collision mesh filename=../meshes/jawpart1_1.stl scale=0.001 0.001 0.001; visual mesh filename=../meshes/jawpart1_1.stl scale=0.001 0.001 0.001
